File: Kicad Files/Bahbahbahbahbah.kicad_pcb (KiCad board)
At the start: 2 copper layers, 31.4 x 35.8 mm, 10 parts, among them U1 AMS1117-3.3, U4 TMR_1-0512, U5 TMR_1-0515, U6 AP7361C-12E

Commit message: bah
Parts:
- added C4: C, Capacitor_SMD:C_0201_0603Metric, F.Cu at (204.7, 78.4)
- added C5: C, Capacitor_SMD:C_0201_0603Metric, F.Cu at (204.7, 80.2)
- J1: renamed from USB-C 5V
- renumbered 1.2V to J2, 3.3V to J3, 12V to J5, 24V to J6, 5V to J7
Routing:
- net GND: track 38.8 -> 48.1 mm
- net Net-(J7-Pin_1): track 52.0 -> 57.7 mm
