File: Kicad Files/Bahbahbahbahbah.kicad_sch (KiCad schematic)
At the start: 12 parts, among them J1 USB_C_Receptacle_PowerOnly_6P, J2 Conn_01x02_Socket, J3 Conn_01x02_Socket, J5 Conn_01x02_Socket, J6 Conn_01x02_Socket, J7 Conn_01x02_Socket, U1 AMS1117-3.3, U4 TMR_1-0512, U5 TMR_1-0515, U6 AP7361C-12E

Commit message: bah
Parts:
- C4, C5: footprint (none) -> Capacitor_SMD:C_0201_0603Metric
Changed lines of the file:
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@@
 			)
 		)
-		(property "Footprint" ""
+		(property "Footprint" "Capacitor_SMD:C_0201_0603Metric"
 			(at 99.06 89.2048 0)
 			(hide yes)
@@
 			)
 		)
-		(property "Footprint" ""
+		(property "Footprint" "Capacitor_SMD:C_0201_0603Metric"
 			(at 97.79 61.2648 0)
 			(hide yes)
